File: Electronics/virtual_clues/virtual_clues.sch (KiCad schematic (older format))
At the start: 10 parts, among them J1 TempSensor, Q1 IRLB8721PBF

Commit message: ordered PCB & complete class based re-write
Parts:
- removed A1: Arduino_Nano, Module:Arduino_Nano_WithMountingHoles, symbol MCU_Module:Arduino_Nano_v3.x
- removed J1: TempSensor, symbol Connector:Screw_Terminal_01x03
- removed J?: heatLED, symbol Connector:Screw_Terminal_01x02
- removed Q1: IRLB8721PBF, Package_TO_SOT_THT:TO-220-3_Vertical, symbol Transistor_FET:IRLB8721PBF
- removed heatMat, mouseTemp: mouseTemp, symbol Connector:Screw_Terminal_01x02
- removed led_res_1: 560, symbol Device:R
- removed led_res_2: 150, symbol Device:R
- removed powerLed1: green, symbol Device:LED
- removed refResistor1: 10k, symbol Device:R
